File: M130-Distribution-HUB.kicad_pcb (KiCad board)
At the start: 4 copper layers, 152.4 x 114.3 mm, 23 parts, among them CN0 6437288-3

Commit message: slight board update
Other:
- board text added: "10A"
- board text removed: "30A"
